File: FSNS_APPS_2025.kicad_pcb (KiCad board)
At the start: 2 copper layers, 89 x 60 mm, 73 parts, among them J1 Conn_01x04_Pin, J2 Conn_01x03_Pin, J3 Conn_01x03_Pin, J4 Conn_01x04_Pin, J5 Conn_01x08_Pin, K1 PR12-12V-360-1A, Q1 NDT3055L, SW1 SW_Push, U1 STM32F103C8T6, U2 MCP6001-OT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

Commit message: Fixed unconnected footprints
Routing:
- net +3.3VA: track 29.5 -> 35.9 mm, vias 4 -> 6
- net Net-(U2--): track 14.0 -> 15.2 mm
Changed lines of the file:
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@@
 		(tags "capacitor")
 		(property "Reference" "C12"
-			(at -0.25 -1.75 90)
+			(at 1.6125 -1.75 90)
 			(layer "F.SilkS")
 			(effects
@@
 	)
 	(segment
+		(start 184.3375 57.75)
+		(end 182.27 57.75)
+		(width 0.3)
+		(layer "F.Cu")
+		(net 2)
+	)
+	(segment
 		(start 194.25 82.25)
 		(end 193.5 82.25)
@@
 	)
 	(segment
-		(start 184.75 61.75)
-		(end 184.75 61)
-		(width 0.5)
-		(layer "F.Cu")
-		(net 2)
-	)
-	(segment
 		(start 197 50.75)
 		(end 195.808505 50.75)
@@
 	)
 	(segment
-		(start 184.3375 57.75)
-		(end 182.27 57.75)
-		(width 0.3)
-		(layer "F.Cu")
-		(net 2)
-	)
-	(segment
 		(start 171.5 60.775)
 		(end 172.225 60.775)
@@
 	)
 	(segment
+		(start 184.252 62.724)
+		(end 184.252 61.002)
+		(width 0.5)
+		(layer "F.Cu")
+		(net 2)
+	)
+	(segment
+		(start 182 58.02)
+		(end 180.77 58.02)
+		(width 0.3)
+		(layer "F.Cu")
+		(net 2)
+	)
+	(segment
 		(start 161.5 36.75)
 		(end 160 38.25)
@@
 	)
 	(segment
+		(start 180.77 58.02)
+		(end 180.75 58)
+		(width 0.3)
+		(layer "F.Cu")
+		(net 2)
+	)
+	(segment
 		(start 212.25 69.25)
 		(end 212.25 68.5)
@@
 	)
 	(segment
-		(start 183.75 61.75)
-		(end 183.75 61)
-		(width 0.5)
-		(layer "F.Cu")
-		(net 2)
-	)
-	(segment
 		(start 226.787502 47.5)
 		(end 226.7875 47.499998)
@@
 	)
 	(segment
-		(start 184.252 62.248)
-		(end 184.75 61.75)
-		(width 0.5)
-		(layer "F.Cu")
-		(net 2)
-	)
-	(segment
 		(start 196 54.5)
 		(end 195.52 54.98)
@@
 	)
 	(segment
-		(start 184.252 62.252)
-		(end 183.75 61.75)
-		(width 0.5)
-		(layer "F.Cu")
-		(net 2)
-	)
-	(segment
 		(start 228.75 69.25)
 		(end 228.75 68.5)
@@
 	)
 	(segment
+		(start 182.27 57.75)
+		(end 182 58.02)
+		(width 0.3)
+		(layer "F.Cu")
+		(net 2)
+	)
+	(segment
 		(start 229.75 69.25)
 		(end 229.75 68.5)
@@
 	)
 	(segment
-		(start 182.27 57.75)
-		(end 182 58.02)
-		(width 0.3)
-		(layer "F.Cu")
-		(net 2)
-	)
-	(segment
 		(start 213.182 82.75)
 		(end 213.182 81.75)
@@
 	)
 	(via
-		(at 183.75 61)
+		(at 226.432 76.25)
 		(size 0.6)
 		(drill 0.3)
@@
 	)
 	(via
-		(at 226.432 76.25)
+		(at 197 50.75)
 		(size 0.6)
 		(drill 0.3)
@@
 	)
 	(via
-		(at 197 50.75)
+		(at 211.932 79)
 		(size 0.6)
 		(drill 0.3)
@@
 	)
 	(via
-		(at 211.932 79)
+		(at 188.5 68)
 		(size 0.6)
 		(drill 0.3)
@@
 	)
 	(via
-		(at 188.5 68)
+		(at 184.25 61)
 		(size 0.6)
 		(drill 0.3)
 		(layers "F.Cu" "B.Cu")
-		(free yes)
 		(net 2)
 	)
@@
 	)
 	(via
+		(at 180.75 58)
+		(size 0.6)
+		(drill 0.3)
+		(layers "F.Cu" "B.Cu")
+		(free yes)
+		(net 2)
+	)
+	(via
 		(at 224.5 61.5)
 		(size 0.6)
@@
 	)
 	(via
-		(at 184.75 61)
-		(size 0.6)
-		(drill 0.3)
-		(layers "F.Cu" "B.Cu")
-		(free yes)
-		(net 2)
-	)
-	(via
 		(at 213.182 82.75)
 		(size 0.6)
@@
 	)
 	(segment
+		(start 209.75 44.3425)
+		(end 209.75 45)
+		(width 0.5)
+		(layer "F.Cu")
+		(net 3)
+	)
+	(segment
 		(start 202.75 45.25)
 		(end 202.75 44.23)
@@
 	)
 	(segment
+		(start 209.75 45)
+		(end 209.75 45.5)
+		(width 0.5)
+		(layer "F.Cu")
+		(net 3)
+	)
+	(segment
 		(start 195.75 53.02)
 		(end 194.75 54.02)
@@
 	)
 	(segment
+		(start 207.75 44.25)
+		(end 205 44.25)
+		(width 0.5)
+		(layer "F.Cu")
+		(net 3)
+	)
+	(segment
 		(start 212.25 45.5)
 		(end 212.25 44.934816)
@@
 	)
 	(via
+		(at 209.75 45.5)
+		(size 0.6)
+		(drill 0.3)
+		(layers "F.Cu" "B.Cu")
+		(net 3)
+	)
+	(via
 		(at 202.75 45.25)
 		(size 0.6)
@@
 		(net 3)
 	)
+	(via
+		(at 207.75 44.25)
+		(size 0.6)
+		(drill 0.3)
+		(layers "F.Cu" "B.Cu")
+		(net 3)
+	)
 	(segment
 		(start 202.75 45.25)
@@
 	)
 	(segment
+		(start 209.75 45.5)
+		(end 209 45.5)
+		(width 0.5)
+		(layer "B.Cu")
+		(net 3)
+	)
+	(segment
+		(start 209 45.5)
+		(end 207.75 44.25)
+		(width 0.5)
+		(layer "B.Cu")
+		(net 3)
+	)
+	(segment
 		(start 193 50)
 		(end 195.75 52.75)
@@
 	)
 	(segment
+		(start 213.2 42.2)
+		(end 212 41)
+		(width 0.3)
+		(layer "F.Cu")
+		(net 52)
+	)
+	(segment
 		(start 213.2 43.225)
 		(end 213.2 42.2)
@@
 	(segment
 		(start 208.75 42.5)
-		(end 208.75 45)
+		(end 208.75 46)
 		(width 0.3)
 		(layer "F.Cu")
@@
 	)
 	(segment
-		(start 208.75 45)
-		(end 209.25 45.5)
+		(start 209 46.25)
+		(end 210.55 46.25)
 		(width 0.3)
 		(layer "F.Cu")
@@
 	)
 	(segment
-		(start 209.25 45.5)
+		(start 210.55 46.25)
 		(end 211.3 45.5)
 		(width 0.3)
@@
 	)
 	(segment
+		(start 211.26 47.25)
+		(end 211.26 45.204598)
+		(width 0.5)
+		(layer "F.Cu")
+		(net 52)
+	)
+	(segment
 		(start 210.25 41)
 		(end 208.75 42.5)
@@
 	)
 	(segment
-		(start 211.26 47.25)
-		(end 211.26 45.204598)
+		(start 211.26 45.54)
+		(end 211.3 45.5)
 		(width 0.5)
 		(layer "F.Cu")
@@
 	)
 	(segment
-		(start 213.2 42.2)
-		(end 212 41)
+		(start 208.75 46)
+		(end 209 46.25)
 		(width 0.3)
 		(layer "F.Cu")
@@
 		(layer "F.Cu")
 		(net 52)
-	)
-	(segment
-		(start 211.26 45.54)
-		(end 211.3 45.5)
-		(width 0.5)
-		(layer "F.Cu")
-		(net 52)
